Commit message: Imported upstream version '0.2.0' of 'upstream'

File: flir_ptu_description/urdf/d46.urdf.xacro (robot description, xacro)
@@ -1,5 +1,4 @@
 <?xml version="1.0"?>
-<robot name="ptu_d46"
-       xmlns:xacro="http://ros.org/wiki/xacro">
+<robot name="ptu_d46" xmlns:xacro="http://www.ros.org/wiki/xacro">
   <xacro:property name="pan_velocity" value="1.0" />
   <xacro:property name="pan_range" value="2.775" />
@@ -11,37 +10,68 @@
                params="ptu_name joint_name">
     <link name="${ptu_name}_${joint_name}_link">
-      <!-- <inertial>
+      <inertial>
         <mass value="0.65" />
-        <inertia ... ? />
-      </inertial> -->
+        <origin xyz="0 0 0" rpy="0 0 0" />
+        <inertia ixx="0.0001" ixy="0" ixz="0" iyy="0.0001" iyz="0" izz="0.0001" />
+      </inertial>
       <visual>
         <material name="ptu_body_color">
           <color rgba="0.3 0.3 0.3 1.0" />
         </material>
+        <origin xyz="-0.0295 0.011 0" rpy="3.14 0 0" />
+        <geometry>
+          <mesh filename="package://flir_ptu_description/meshes/flir-ptu-simple.stl"/>
+        </geometry>
+      </visual>
+      <collision>
         <geometry>
           <box size="0.045 0.065 0.044" />
         </geometry>
         <origin xyz="0 0.011 0" />
-      </visual>
-      <visual>
+      </collision>
+      <collision>
         <geometry>
           <box size="0.046 0.044 0.044" />
         </geometry>
         <origin xyz="-0.045 0.0215 0" />
-      </visual>
-      <visual>
+      </collision>
+      <collision>
         <geometry>
           <cylinder length="0.015" radius="0.005" />
         </geometry>
         <origin xyz="-0.074 0.021 0" rpy="0 1.57 0" />
-      </visual>
+      </collision>
     </link>
+    <gazebo reference="${ptu_name}_${joint_name}_link">
+        <material>Gazebo/DarkGrey</material>
+    </gazebo>
   </xacro:macro>
-  <xacro:macro name="ptu_d46" params="name">
+  <xacro:macro name="d46_transmission" params="name">
+    <transmission name="${name}_trans">
+      <type>transmission_interface/SimpleTransmission</type>
+      <joint name="${name}">
+        <hardwareInterface>PositionJointInterface</hardwareInterface>
+      </joint>
+      <actuator name="${name}_motor">
+        <mechanicalReduction>1</mechanicalReduction>
+      </actuator>
+    </transmission>
+  </xacro:macro>
+  <xacro:macro name="ptu_d46" params="name pan_offset:=0.0">
     <d46_stepper_module ptu_name="${name}" joint_name="pan" />
     <d46_stepper_module ptu_name="${name}" joint_name="tilt" />
-    <link name="${name}_base_link" />
-    <link name="${name}_tilted_link" />
-    <link name="${name}_mount_link" />
+    <link name="${name}_base_link">
+       <inertial>
+            <mass value="2e-06"/>
+            <inertia ixx="1.1e-09" ixy="0" ixz="0" iyy="1.1e-09" iyz="0" izz="1.1e-09"/>
+        </inertial>
+    </link>
+    <link name="${name}_tilted_link"/>
+    <link name="${name}_mount_link">
+        <inertial>
+            <mass value="2e-06"/>
+            <inertia ixx="1.1e-09" ixy="0" ixz="0" iyy="1.1e-09" iyz="0" izz="1.1e-09"/>
+        </inertial>
+    </link>
     <!-- There's an offset between the origin of the pan joint and the origin of
          the overall device, which is between the mounting screws on its base. -->
@@ -54,10 +84,11 @@
     <joint name="${name}_pan" type="revolute">
       <parent link="${name}_pan_link" />
-      <origin xyz="0 0 0.066" rpy="-1.5708 0 0" />
+      <origin xyz="0 0 0.066" rpy="-1.5708 0 ${pan_offset}" />
       <child link="${name}_tilt_link" />
-      <axis xyz="0 1 0" rpy="0 0 0" />
-      <limit lower="${pan_range}" upper="${-pan_range}"
+      <axis xyz="0 -1 0" rpy="3.14159 0 0" />
+      <limit lower="${-pan_range}" upper="${pan_range}"
              effort="${joint_effort}" velocity="${pan_velocity}" />
     </joint>
+    <d46_transmission name="${name}_pan" />
     <!-- The tilt joint -->
     <joint name="${name}_tilt" type="revolute">
@@ -69,4 +100,5 @@
              effort="${joint_effort}" velocity="${tilt_velocity}" />
     </joint>
+    <d46_transmission name="${name}_tilt" />
     <!-- Fixed joint to provide a convenient attachment point for accessories. -->
     <joint name="${name}_mount" type="fixed">

File: flir_ptu_description/urdf/example.urdf.xacro (robot description, xacro)
@@ -1,5 +1,5 @@
 <?xml version="1.0"?>
 <robot name="ptu_d46"
-       xmlns:xacro="http://ros.org/wiki/xacro">
+       xmlns:xacro="http://www.ros.org/wiki/xacro">
   <link name="base_link" />
   <!-- Include and invoke the macro which creates a D46 -->

Commit message: Imported upstream version '0.2.1' of 'upstream'

File: flir_ptu_description/urdf/d46.urdf.xacro (robot description, xacro)
@@ -7,44 +7,4 @@
   <xacro:property name="tilt_down_range" value="0.82" />
   <xacro:property name="joint_effort" value="30" />
-  <xacro:macro name="d46_stepper_module"
-               params="ptu_name joint_name">
-    <link name="${ptu_name}_${joint_name}_link">
-      <inertial>
-        <mass value="0.65" />
-        <origin xyz="0 0 0" rpy="0 0 0" />
-        <inertia ixx="0.0001" ixy="0" ixz="0" iyy="0.0001" iyz="0" izz="0.0001" />
-      </inertial>
-      <visual>
-        <material name="ptu_body_color">
-          <color rgba="0.3 0.3 0.3 1.0" />
-        </material>
-        <origin xyz="-0.0295 0.011 0" rpy="3.14 0 0" />
-        <geometry>
-          <mesh filename="package://flir_ptu_description/meshes/flir-ptu-simple.stl"/>
-        </geometry>
-      </visual>
-      <collision>
-        <geometry>
-          <box size="0.045 0.065 0.044" />
-        </geometry>
-        <origin xyz="0 0.011 0" />
-      </collision>
-      <collision>
-        <geometry>
-          <box size="0.046 0.044 0.044" />
-        </geometry>
-        <origin xyz="-0.045 0.0215 0" />
-      </collision>
-      <collision>
-        <geometry>
-          <cylinder length="0.015" radius="0.005" />
-        </geometry>
-        <origin xyz="-0.074 0.021 0" rpy="0 1.57 0" />
-      </collision>
-    </link>
-    <gazebo reference="${ptu_name}_${joint_name}_link">
-        <material>Gazebo/DarkGrey</material>
-    </gazebo>
-  </xacro:macro>
   <xacro:macro name="d46_transmission" params="name">
     <transmission name="${name}_trans">
@@ -59,6 +19,50 @@
   </xacro:macro>
   <xacro:macro name="ptu_d46" params="name pan_offset:=0.0">
-    <d46_stepper_module ptu_name="${name}" joint_name="pan" />
-    <d46_stepper_module ptu_name="${name}" joint_name="tilt" />
+    <link name="${name}_tilt_link">
+      <inertial>
+        <mass value="0.65" />
+        <origin xyz="0 0 0" rpy="0 0 0" />
+        <inertia ixx="0.0001" ixy="0" ixz="0" iyy="0.0001" iyz="0" izz="0.0001" />
+      </inertial>
+      <visual>
+        <material name="ptu_body_color">
+          <color rgba="0.3 0.3 0.3 1.0" />
+        </material>
+        <geometry>
+          <mesh filename="package://flir_ptu_description/meshes/flir-ptu-tilt-motor.stl"/>
+        </geometry>
+      </visual>
+      <collision>
+        <geometry>
+          <mesh filename="package://flir_ptu_description/meshes/flir-ptu-tilt-motor-collision.stl"/>
+        </geometry>
+      </collision>
+    </link>
+    <gazebo reference="${name}_tilt_link">
+        <material>Gazebo/DarkGrey</material>
+    </gazebo>
+    <link name="${name}_pan_link">
+      <inertial>
+        <mass value="0.65" />
+        <origin xyz="0 0 0" rpy="0 0 0" />
+        <inertia ixx="0.0001" ixy="0" ixz="0" iyy="0.0001" iyz="0" izz="0.0001" />
+      </inertial>
+      <visual>
+        <material name="ptu_body_color">
+          <color rgba="0.3 0.3 0.3 1.0" />
+        </material>
+        <geometry>
+          <mesh filename="package://flir_ptu_description/meshes/flir-ptu-pan-motor.stl"/>
+        </geometry>
+      </visual>
+      <collision>
+        <geometry>
+          <mesh filename="package://flir_ptu_description/meshes/flir-ptu-pan-motor-collision.stl"/>
+        </geometry>
+      </collision>
+    </link>
+    <gazebo reference="${name}_pan_link">
+        <material>Gazebo/DarkGrey</material>
+    </gazebo>
     <link name="${name}_base_link">
        <inertial>
@@ -67,5 +71,19 @@
         </inertial>
     </link>
-    <link name="${name}_tilted_link"/>
+    <link name="${name}_tilted_link">
+      <visual>
+        <material name="ptu_body_color">
+          <color rgba="0.3 0.3 0.3 1.0" />
+        </material>
+        <geometry>
+          <mesh filename="package://flir_ptu_description/meshes/flir-ptu-camera-mount.stl"/>
+        </geometry>
+      </visual>
+      <collision>
+        <geometry>
+          <mesh filename="package://flir_ptu_description/meshes/flir-ptu-camera-mount.stl"/>
+        </geometry>
+      </collision>
+    </link>
     <link name="${name}_mount_link">
         <inertial>
@@ -74,15 +92,13 @@
         </inertial>
     </link>
-    <!-- There's an offset between the origin of the pan joint and the origin of
-         the overall device, which is between the mounting screws on its base. -->
     <joint name="${name}_base" type="fixed">
       <parent link="${name}_base_link"/>
       <child link="${name}_pan_link"/>
-      <origin xyz="0 -0.011 0.022"/>
+      <origin xyz="0 0 0"/>
     </joint>
     <!-- The pan joint -->
     <joint name="${name}_pan" type="revolute">
       <parent link="${name}_pan_link" />
-      <origin xyz="0 0 0.066" rpy="-1.5708 0 ${pan_offset}" />
+      <origin xyz="0 -0.00955 0.046774" rpy="-1.5708 0 ${pan_offset}" />
       <child link="${name}_tilt_link" />
       <axis xyz="0 -1 0" rpy="3.14159 0 0" />
@@ -90,9 +106,9 @@
              effort="${joint_effort}" velocity="${pan_velocity}" />
     </joint>
-    <d46_transmission name="${name}_pan" />
+    <xacro:d46_transmission name="${name}_pan" />
     <!-- The tilt joint -->
     <joint name="${name}_tilt" type="revolute">
       <parent link="${name}_tilt_link" />
-      <origin xyz="0 0 0" rpy="-1.5708 0 0" />
+      <origin xyz="0 -0.043713 0" rpy="-1.5708 0 0" />
       <child link="${name}_tilted_link" />
       <axis xyz="0 1 0" />
@@ -100,10 +116,10 @@
              effort="${joint_effort}" velocity="${tilt_velocity}" />
     </joint>
-    <d46_transmission name="${name}_tilt" />
+    <xacro:d46_transmission name="${name}_tilt" />
     <!-- Fixed joint to provide a convenient attachment point for accessories. -->
     <joint name="${name}_mount" type="fixed">
       <parent link="${name}_tilted_link"/>
       <child link="${name}_mount_link"/>
-      <origin xyz="0 0 -0.03912" rpy="3.1416 0 0" />
+      <origin xyz="0 0 -0.039116" rpy="3.1416 0 0" />
     </joint>
   </xacro:macro>

File: flir_ptu_description/urdf/example.urdf.xacro (robot description, xacro)
@@ -5,5 +5,5 @@
   <!-- Include and invoke the macro which creates a D46 -->
   <xacro:include filename="d46.urdf.xacro" />
-  <ptu_d46 name="ptu" />
+  <xacro:ptu_d46 name="ptu" />
   <!-- Create a fixed joint to connect the PTU to the rest of the robot -->
   <joint name="base_to_ptu_base" type="fixed">
